Commit message: modified rplidar laser frame orientation

File: clearpath_common/clearpath_sensors_description/urdf/rplidar.urdf.xacro (robot description, xacro)
@@ -53,5 +53,5 @@
       <parent link="${name}_link" />
       <child link="${name}_laser" />
-      <origin xyz="0 0 0.034" rpy="0 0 0"/>
+      <origin xyz="0 0 0.034" rpy="0 0 3.141592653589793"/>
     </joint>
     <xacro:property name="samples" value="${round((max_ang - min_ang) * 180 / (ang_res * pi))}"/>
