Commit message: fixing rplidar integration

File: husky_commander/config/husky_basic/robot.urdf.xacro (robot description, xacro)
@@ -22,17 +22,14 @@
   <!-- Mounts -->
   <!-- Sensors -->
-  <xacro:include filename="$(find clearpath_platform_description)/urdf/a200/attachments/rplidar.urdf.xacro"/>
-  <xacro:rplidar
-      name="front_rplidar"
-      parent_link="front_bumper_link"
-      xyz="0.0 0.0 0.08"
-      rpy="0 0 0"
-      laser_rpy="0 0 ${-M_PI/2}"/>
-  <xacro:rplidar
-      name="rear_rplidar"
-      parent_link="rear_bumper_link"
-      xyz="0.0 0.0 0.08"
-      rpy="0 0 ${M_PI}"
-      laser_rpy="0 0 ${-M_PI/2}"/>
+  <!-- lidar2d_0 -->
+  <xacro:include filename="$(find clearpath_sensors_description)/urdf/rplidar.urdf.xacro"/>
+  <xacro:rplidar name="lidar2d_0" parent_link="front_bumper_link" ang_res="0.5" min_ang="-3.141592653589793" max_ang="3.141592653589793" min_range="0.05" max_range="25.0" update_rate="50">
+    <origin xyz="0.0 0.0 0.08" rpy="0.0 0.0 0.0"/>
+  </xacro:rplidar>
+  <!-- lidar2d_1 -->
+  <xacro:include filename="$(find clearpath_sensors_description)/urdf/rplidar.urdf.xacro"/>
+  <xacro:rplidar name="lidar2d_1" parent_link="rear_bumper_link" ang_res="0.5" min_ang="-3.141592653589793" max_ang="3.141592653589793" min_range="0.05" max_range="25.0" update_rate="50">
+    <origin xyz="0.0 0.0 0.08" rpy="0.0 0.0 3.141592653589793"/>
+  </xacro:rplidar>
   <!-- Manipulators -->
   <!-- Extras -->

Commit message: adding imu sensor for simulation

File: husky_commander/config/husky_basic/robot.urdf.xacro (robot description, xacro)
@@ -32,4 +32,9 @@
     <origin xyz="0.0 0.0 0.08" rpy="0.0 0.0 3.141592653589793"/>
   </xacro:rplidar>
+  <!-- imu_0 -->
+  <xacro:include filename="$(find clearpath_sensors_description)/urdf/microstrain_imu.urdf.xacro"/>
+  <xacro:microstrain_imu name="imu_0" parent_link="base_link" update_rate="100">
+    <origin xyz="0.0 0.0 0.05" rpy="0.0 0.0 0.0"/>
+  </xacro:microstrain_imu>
   <!-- Manipulators -->
   <!-- Extras -->
